File: output/pcbs/corne_pcb.kicad_pcb (KiCad board)
At the start: 2 copper layers, 164.2 x 123.2 mm, 80 parts

Commit message: update2
Parts:
- added LED1: , ceoloide:led_SK6812mini-e (per-key, reversible), B.Cu at (152.4, 145.0)
- added LED10: , ceoloide:led_SK6812mini-e (per-key, reversible), B.Cu at (171.4, 69.0)
- added LED11: , ceoloide:led_SK6812mini-e (per-key, reversible), B.Cu at (190.4, 140.2)
- added LED12: , ceoloide:led_SK6812mini-e (per-key, reversible), B.Cu at (190.4, 121.2)
- added LED13: , ceoloide:led_SK6812mini-e (per-key, reversible), B.Cu at (190.4, 102.2)
- added LED14: , ceoloide:led_SK6812mini-e (per-key, reversible), B.Cu at (190.4, 83.2)
- added LED15: , ceoloide:led_SK6812mini-e (per-key, reversible), B.Cu at (190.4, 64.2)
- added LED16: , ceoloide:led_SK6812mini-e (per-key, reversible), B.Cu at (209.4, 137.9)
- added LED17: , ceoloide:led_SK6812mini-e (per-key, reversible), B.Cu at (209.4, 118.9)
- added LED18: , ceoloide:led_SK6812mini-e (per-key, reversible), B.Cu at (209.4, 99.9)
- added LED19: , ceoloide:led_SK6812mini-e (per-key, reversible), B.Cu at (209.4, 80.9)
- added LED2: , ceoloide:led_SK6812mini-e (per-key, reversible), B.Cu at (150.0, 126.0)
- added LED20: , ceoloide:led_SK6812mini-e (per-key, reversible), B.Cu at (209.4, 61.9)
- added LED21: , ceoloide:led_SK6812mini-e (per-key, reversible), B.Cu at (228.4, 121.2)
- added LED22: , ceoloide:led_SK6812mini-e (per-key, reversible), B.Cu at (228.4, 102.2)
- added LED23: , ceoloide:led_SK6812mini-e (per-key, reversible), B.Cu at (228.4, 83.2)
- added LED24: , ceoloide:led_SK6812mini-e (per-key, reversible), B.Cu at (228.4, 64.2)
- added LED25: , ceoloide:led_SK6812mini-e (per-key, reversible), B.Cu at (247.4, 123.6)
- added LED26: , ceoloide:led_SK6812mini-e (per-key, reversible), B.Cu at (247.4, 104.6)
- added LED27: , ceoloide:led_SK6812mini-e (per-key, reversible), B.Cu at (247.4, 85.6)
- added LED28: , ceoloide:led_SK6812mini-e (per-key, reversible), B.Cu at (247.4, 66.6)
- added LED29: , ceoloide:led_SK6812mini-e (per-key, reversible), B.Cu at (261.4, 104.9)
- added LED3: , ceoloide:led_SK6812mini-e (per-key, reversible), B.Cu at (150.0, 107.0)
- added LED30: , ceoloide:led_SK6812mini-e (per-key, reversible), B.Cu at (266.4, 76.1)
- added LED31: , ceoloide:led_SK6812mini-e (per-key, reversible), B.Cu at (239.2, 142.8)
- added LED32: , ceoloide:led_SK6812mini-e (per-key, reversible), B.Cu at (261.2, 153.8)
- added LED33: , ceoloide:led_SK6812mini-e (per-key, reversible), B.Cu at (266.2, 135.0)
- added LED34: , ceoloide:led_SK6812mini-e (per-key, reversible), B.Cu at (277.6, 163.3)
- added LED35: , ceoloide:led_SK6812mini-e (per-key, reversible), B.Cu at (282.7, 144.5)
- added LED4: , ceoloide:led_SK6812mini-e (per-key, reversible), B.Cu at (150.0, 88.0)
- added LED5: , ceoloide:led_SK6812mini-e (per-key, reversible), B.Cu at (150.0, 69.0)
- added LED6: , ceoloide:led_SK6812mini-e (per-key, reversible), B.Cu at (171.4, 145.0)
- added LED7: , ceoloide:led_SK6812mini-e (per-key, reversible), B.Cu at (171.4, 126.0)
- added LED8: , ceoloide:led_SK6812mini-e (per-key, reversible), B.Cu at (171.4, 107.0)
- added LED9: , ceoloide:led_SK6812mini-e (per-key, reversible), B.Cu at (171.4, 88.0)
Routing:
- net (no net): track 112.6 -> 586.0 mm, vias 0 -> 70
- net VCC: track 0.00 -> 131.4 mm, vias 0 -> 35
- net GND: track 0.00 -> 131.4 mm, vias 0 -> 35
